File: IS31FL3731_ssop28_dip.kicad_pcb (KiCad board)
At the start: 2 copper layers, 19 x 41.8 mm, 15 parts, among them J1 Conn_01x07, U1 IS31FL3731

Commit message: Fix labels
Other:
- board text added: "+5V"
- board text added: "CA1"
- board text added: "CB1"
Changed lines of the file:
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@@
   (general
     (thickness 1.6)
-    (drawings 10)
+    (drawings 14)
     (tracks 198)
     (zones 0)
@@
   )
   (setup
-    (last_trace_width 0.2)
+    (last_trace_width 0.154)
     (user_trace_width 0.2)
     (user_trace_width 0.25)
@@
     (tags resistor)
     (attr smd)
-    (fp_text reference R_EXT1 (at 0.635 -1.905 270) (layer B.SilkS)
+    (fp_text reference R_EXT1 (at -0.98552 -1.67132 270) (layer B.SilkS)
       (effects (font (size 1 1) (thickness 0.15)) (justify mirror))
     )
@@
     (tags resistor)
     (attr smd)
-    (fp_text reference R3 (at 2.67 0.31) (layer B.SilkS)
+    (fp_text reference R3 (at 2.78638 0.07874) (layer B.SilkS)
       (effects (font (size 1 1) (thickness 0.15)) (justify mirror))
     )
@@
     (tags resistor)
     (attr smd)
-    (fp_text reference R2 (at -2.54 0 90) (layer B.SilkS)
+    (fp_text reference R2 (at 0.1778 -1.42494 90) (layer B.SilkS)
       (effects (font (size 1 1) (thickness 0.15)) (justify mirror))
     )
@@
     (tags resistor)
     (attr smd)
-    (fp_text reference R_AD1 (at 2.49 0) (layer B.SilkS)
+    (fp_text reference R_AD1 (at -2.1336 1.65354) (layer B.SilkS)
       (effects (font (size 1 1) (thickness 0.15)) (justify mirror))
     )
@@
     (descr "Through hole straight pin header, 1x07, 2.54mm pitch, single row")
     (tags "Through hole pin header THT 1x07 2.54mm single row")
-    (fp_text reference J1 (at 2.07 -1.36) (layer B.SilkS)
+    (fp_text reference J1 (at 2.311 -0.169) (layer B.SilkS)
       (effects (font (size 1 1) (thickness 0.15)) (justify mirror))
     )
@@
     (tags capacitor)
     (attr smd)
-    (fp_text reference C2 (at -2.54 0 90) (layer B.SilkS)
+    (fp_text reference C2 (at 0 1.74498 90) (layer B.SilkS)
       (effects (font (size 1 1) (thickness 0.15)) (justify mirror))
     )
@@
     )
   )
-  (gr_text AUDIO (at 121.793 88.922) (layer F.SilkS)
-    (effects (font (size 0.5 0.5) (thickness 0.125)))
-  )
-  (gr_text SCL (at 121.3 93.875) (layer F.SilkS)
-    (effects (font (size 0.5 0.5) (thickness 0.125)))
+  (gr_text CB1 (at 131.5716 122.005) (layer F.SilkS)
+    (effects (font (size 1 1) (thickness 0.15)))
+  )
+  (gr_text CA1 (at 122.2244 101.7104) (layer F.SilkS)
+    (effects (font (size 1 1) (thickness 0.15)))
+  )
+  (gr_text +5V (at 121.8688 99.0434) (layer F.SilkS)
+    (effects (font (size 1 1) (thickness 0.15)))
+  )
+  (gr_text GND (at 122.1228 96.6304) (layer F.SilkS)
+    (effects (font (size 1 1) (thickness 0.15)))
+  )
+  (gr_text AUDIO (at 122.961 88.8834) (layer F.SilkS)
+    (effects (font (size 1 1) (thickness 0.15)))
+  )
+  (gr_text SCL (at 122.2752 93.8618) (layer F.SilkS)
+    (effects (font (size 1 1) (thickness 0.15)))
   )
   (gr_text GND (at 125.56336 105.01444 90) (layer B.SilkS)
     (effects (font (size 0.5 0.5) (thickness 0.125)) (justify mirror))
   )
-  (gr_text SDA (at 121.412 91.44) (layer F.SilkS)
-    (effects (font (size 0.5 0.5) (thickness 0.125)))
-  )
-  (gr_text ~INTB (at 121.666 86.487) (layer F.SilkS)
-    (effects (font (size 0.5 0.5) (thickness 0.125)))
-  )
-  (gr_text ~SHUTDOWN (at 122.8 83.947) (layer F.SilkS)
-    (effects (font (size 0.5 0.5) (thickness 0.125)))
+  (gr_text SDA (at 122.1482 91.4996) (layer F.SilkS)
+    (effects (font (size 1 1) (thickness 0.15)))
+  )
+  (gr_text ~INTB (at 122.4276 86.4704) (layer F.SilkS)
+    (effects (font (size 1 1) (thickness 0.15)))
+  )
+  (gr_text ~SHUTDOWN (at 124.6882 83.8796) (layer F.SilkS)
+    (effects (font (size 1 1) (thickness 0.15)))
   )
   (gr_line (start 136.5 82) (end 117.5 82) (layer Edge.Cuts) (width 0.05))
